File: dashboard/hw/dash_pcb.sch (KiCad schematic (older format))
At the start: 35 parts, among them J1 LCD, J2 DEBUG, J3 LCD_BL, J4 CAN, J5 POWER, U1 LPC11C24FBD48, U2 TPS62175, U3 TLV70233_SOT23-5, Y1 12MHz

Commit message: more parts shopping
Parts:
- removed J4: CAN, Pin_Headers:Pin_Header_Angled_1x03_Pitch2.54mm, symbol Conn_01x03
- removed J5: POWER, Pin_Headers:Pin_Header_Angled_1x02_Pitch2.00mm, symbol Conn_01x02
- added J4: CAR, Pin_Headers:Pin_Header_Angled_1x06_Pitch2.54mm, symbol Conn_01x06
- added R12: 36, Resistors_SMD:R_1206, symbol R
- J3: footprint Connectors_JST:JST_XH_S03B-XH-A_03x2.50mm_Angled -> Pin_Headers:Pin_Header_Angled_1x03_Pitch2.54mm
- R11: renamed from R?; value 18 -> 36; footprint (none) -> Resistors_SMD:R_1206
- RV1: footprint Potentiometers:Potentiometer_Trimmer_ACP_CA6v_Horizontal -> Potentiometers:Potentiometer_Trimmer_ACP_CA6h_Vertical
Connections:
- net labels added: +BATT
- wire segments 138 -> 109
Other:
- moved on the sheet: C12, C13, C7, R11, R2, R4, Y1

Commit message: add footprint for TI power chip
Parts:
- U2: footprint (none) -> custom_footprints:DQC
Changed lines of the file:
@@
 F 0 "U2" H 1900 650 60  0000 C CNN
 F 1 "TPS62175" H 2150 1100 60  0000 C CNN
-F 2 "" H 2150 1200 60  0001 C CNN
+F 2 "custom_footprints:DQC" H 2150 1200 60  0001 C CNN
 F 3 "https://www.mouser.de/ProductDetail/Texas-Instruments/TPS62175DQCR?qs=sGAEpiMZZMtD8yQon44BRtpT62hWKGFK" H 2150 1200 60  0001 C CNN
 	1    2150 1150

Commit message: add footprint for contrast pot
Parts:
- RV1: footprint Potentiometers:Potentiometer_Trimmer_ACP_CA6h_Vertical -> custom_footprints:Bourns_3362X
Changed lines of the file:
@@
 F 0 "RV1" V 10375 3600 50  0000 C CNN
 F 1 "10k" V 10450 3600 50  0000 C CNN
-F 2 "Potentiometers:Potentiometer_Trimmer_ACP_CA6h_Vertical" H 10550 3600 50  0001 C CNN
+F 2 "custom_footprints:Bourns_3362X" H 10550 3600 50  0001 C CNN
 F 3 "https://www.mouser.de/ProductDetail/Bourns/3362X-1-103LF?qs=sGAEpiMZZMtC25l1F4XBUxECHfqDmxl1ITAi%252bn07c9o%3d" H 10550 3600 50  0001 C CNN
 	1    10550 3600

Commit message: add footprint for inductor
Parts:
- L1: footprint (none) -> custom_footprints:Coilcraft_LPS4018
Changed lines of the file:
@@
 F 0 "L1" V 2800 750 50  0000 C CNN
 F 1 "10u" V 2925 750 50  0000 C CNN
-F 2 "" H 2850 750 50  0001 C CNN
+F 2 "custom_footprints:Coilcraft_LPS4018" H 2850 750 50  0001 C CNN
 F 3 "https://www.mouser.de/ProductDetail/Coilcraft/LPS4018-103MRB?qs=sGAEpiMZZMsg%252by3WlYCkU2oPBW0WnPwqnL16yXxQPg0%3d" H 2850 750 50  0001 C CNN
 	1    2850 750

Commit message: reset automatically when power isn't good
Connections:
- net MCU_~RESET is gone; now on net 5VPG: R7.1, U1.3 (~RESET~/PIO0_0)
Changed lines of the file:
@@
 Connection ~ 1550 1500
 Wire Wire Line
-	2650 1500 2700 1500
+	2650 1500 2950 1500
 Wire Wire Line
 	2700 1500 2700 1550
@@
 	10400 2650 10600 2650
 Connection ~ 10500 2650
+Wire Wire Line
+	2950 1500 2950 1900
+Wire Wire Line
+	2950 1900 3200 1900
+Connection ~ 2700 1500
+Text Label 3200 1900 0    60   ~ 0
+MCU_~RESET
 $EndSCHEMATC

Commit message: lay out power bits
Connections:
- net GND: now also U3.4 (NC)

Commit message: make shrouded version of programming connector
Parts:
- J2: footprint Pin_Headers:Pin_Header_Angled_2x05_Pitch1.27mm -> custom_footprints:Pin_Header_Angled_2x05_Pitch1.27mm_AMPHENOL_SHROUDED
Changed lines of the file:
@@
 F 0 "J2" H 9750 6400 50  0000 C CNN
 F 1 "DEBUG" H 9750 5800 50  0000 C CNN
-F 2 "Pin_Headers:Pin_Header_Angled_2x05_Pitch1.27mm" H 9700 6100 50  0001 C CNN
+F 2 "custom_footprints:Pin_Header_Angled_2x05_Pitch1.27mm_AMPHENOL_SHROUDED" H 9700 6100 50  0001 C CNN
 F 3 "https://www.mouser.de/ProductDetail/Amphenol-FCI/20021512-00010T4LF?qs=sGAEpiMZZMs%252bGHln7q6pmwodwKqstCemugheqdGIyCk%3d" H 9700 6100 50  0001 C CNN
 	1    9700 6100

Commit message: use 4 position connector for car interface
Parts:
- J4: footprint Pin_Headers:Pin_Header_Angled_1x06_Pitch2.54mm -> Pin_Headers:Pin_Header_Angled_1x04_Pitch2.54mm; symbol Conn_01x06 -> Conn_01x04
Connections:
- net CANH: now also J4.3 (Pin_3); no longer J4.6 (Pin_6)
- net CANL: now also J4.4 (Pin_4); no longer J4.5 (Pin_5)
- net GND: no longer J4.3 (Pin_3), J4.4 (Pin_4)
Changed lines of the file:
@@
 $EndComp
 $Comp
-L Conn_01x06 J4
+L Conn_01x04 J4
 U 1 1 5AF30641
-P 10700 1100
+P 10700 1200
 F 0 "J4" H 10700 1400 50  0000 C CNN
-F 1 "CAR" H 10700 700 50  0000 C CNN
-F 2 "Pin_Headers:Pin_Header_Angled_1x06_Pitch2.54mm" H 10700 1100 50  0001 C CNN
-F 3 "https://www.mouser.de/ProductDetail/TE-Connectivity-AMP/281698-6?qs=%2fha2pyFadug9FJ64psl8O%252bSt%252bkgg8uzrxHXiR9bfhg2jsHpVs7%252bIVg%3d%3d" H 10700 1100 50  0001 C CNN
-	1    10700 1100
+F 1 "CAR" H 10700 900 50  0000 C CNN
+F 2 "Pin_Headers:Pin_Header_Angled_1x04_Pitch2.54mm" H 10700 1200 50  0001 C CNN
+F 3 "https://www.mouser.de/ProductDetail/TE-Connectivity-AMP/281698-4?qs=%2fha2pyFadugOWSnGxX0tdzch1lu8VUuW2SzrxAWts0w%3d" H 10700 1200 50  0001 C CNN
+	1    10700 1200
 	1    0    0    1
 $EndComp
-Text Label 10500 800  2    60   ~ 0
+Text Label 10500 1100 2    60   ~ 0
 CANH
-Text Label 10500 900  2    60   ~ 0
+Text Label 10500 1000 2    60   ~ 0
 CANL
 $Comp
 L +BATT #PWR028
 U 1 1 5AF308D1
-P 10250 1250
-F 0 "#PWR028" H 10250 1100 50  0001 C CNN
-F 1 "+BATT" H 10250 1390 50  0000 C CNN
-F 2 "" H 10250 1250 50  0001 C CNN
-F 3 "" H 10250 1250 50  0001 C CNN
-	1    10250 1250
+P 10100 1250
+F 0 "#PWR028" H 10100 1100 50  0001 C CNN
+F 1 "+BATT" H 10100 1390 50  0000 C CNN
+F 2 "" H 10100 1250 50  0001 C CNN
+F 3 "" H 10100 1250 50  0001 C CNN
+	1    10100 1250
 	1    0    0    -1
 $EndComp
@@
 	1650 900  1550 900
 Wire Wire Line
-	1550 900  1550 750
+	1550 750  1550 900
 Connection ~ 1550 750
 Wire Wire Line
@@
 	1150 750  1650 750
 Wire Wire Line
-	10250 1250 10250 1300
-Wire Wire Line
-	10250 1300 10500 1300
-Wire Wire Line
-	10500 1000 10500 1200
-Connection ~ 10500 1100
+	10100 1250 10100 1300
+Wire Wire Line
+	10100 1300 10500 1300
 Wire Wire Line
 	10500 1200 10400 1200
