File: dashboard/hw/dash_pcb.sch (KiCad schematic (older format))
At the start: 36 parts, among them J1 LCD, J2 DEBUG, J3 LCD_BL, J4 CAR, SW1 CONFIG, U1 LPC11C24FBD48, U2 TPS62175, U3 TLV70233_SOT23-5, Y1 12MHz

Commit message: misc changes to part numbers and such
Parts:
- R2, R4, R5, R6, R7: value 60 -> 60.4
Changed lines of the file:
@@
 P 7750 4500
 F 0 "R2" V 7830 4500 50  0000 C CNN
-F 1 "60" V 7750 4500 50  0000 C CNN
+F 1 "60.4" V 7750 4500 50  0000 C CNN
 F 2 "Resistors_SMD:R_0603" V 7680 4500 50  0001 C CNN
-F 3 "https://www.mouser.de/ProductDetail/Yageo/RC0603FR-0759RL?qs=sGAEpiMZZMtlubZbdhIBIHvQf5egq9lvwCJIG56bzdE%3d" H 7750 4500 50  0001 C CNN
+F 3 "https://www.mouser.de/ProductDetail/Bourns/CR0603-FX-60R4ELF?qs=sGAEpiMZZMu61qfTUdNhG6LqqFhkr6pUa8gjAX4b5rM%3d" H 7750 4500 50  0001 C CNN
 	1    7750 4500
 	-1   0    0    1
@@
 P 7950 4500
 F 0 "R4" V 8030 4500 50  0000 C CNN
-F 1 "60" V 7950 4500 50  0000 C CNN
+F 1 "60.4" V 7950 4500 50  0000 C CNN
 F 2 "Resistors_SMD:R_0603" V 7880 4500 50  0001 C CNN
-F 3 "https://www.mouser.de/ProductDetail/Yageo/RC0603FR-0759RL?qs=sGAEpiMZZMtlubZbdhIBIHvQf5egq9lvwCJIG56bzdE%3d" H 7950 4500 50  0001 C CNN
+F 3 "https://www.mouser.de/ProductDetail/Bourns/CR0603-FX-60R4ELF?qs=sGAEpiMZZMu61qfTUdNhG6LqqFhkr6pUa8gjAX4b5rM%3d" H 7950 4500 50  0001 C CNN
 	1    7950 4500
 	-1   0    0    1
@@
 P 10350 5900
 F 0 "R5" V 10430 5900 50  0000 C CNN
-F 1 "60" V 10350 5900 50  0000 C CNN
+F 1 "60.4" V 10350 5900 50  0000 C CNN
 F 2 "Resistors_SMD:R_0603" V 10280 5900 50  0001 C CNN
-F 3 "https://www.mouser.de/ProductDetail/Yageo/RC0603FR-0759RL?qs=sGAEpiMZZMtlubZbdhIBIHvQf5egq9lvwCJIG56bzdE%3d" H 10350 5900 50  0001 C CNN
+F 3 "https://www.mouser.de/ProductDetail/Bourns/CR0603-FX-60R4ELF?qs=sGAEpiMZZMu61qfTUdNhG6LqqFhkr6pUa8gjAX4b5rM%3d" H 10350 5900 50  0001 C CNN
 	1    10350 5900
 	0    -1   -1   0
@@
 P 10350 6000
 F 0 "R6" V 10430 6000 50  0000 C CNN
-F 1 "60" V 10350 6000 50  0000 C CNN
+F 1 "60.4" V 10350 6000 50  0000 C CNN
 F 2 "Resistors_SMD:R_0603" V 10280 6000 50  0001 C CNN
-F 3 "https://www.mouser.de/ProductDetail/Yageo/RC0603FR-0759RL?qs=sGAEpiMZZMtlubZbdhIBIHvQf5egq9lvwCJIG56bzdE%3d" H 10350 6000 50  0001 C CNN
+F 3 "https://www.mouser.de/ProductDetail/Bourns/CR0603-FX-60R4ELF?qs=sGAEpiMZZMu61qfTUdNhG6LqqFhkr6pUa8gjAX4b5rM%3d" H 10350 6000 50  0001 C CNN
 	1    10350 6000
 	0    1    1    0
@@
 P 10350 6300
 F 0 "R7" V 10430 6300 50  0000 C CNN
-F 1 "60" V 10350 6300 50  0000 C CNN
+F 1 "60.4" V 10350 6300 50  0000 C CNN
 F 2 "Resistors_SMD:R_0603" V 10280 6300 50  0001 C CNN
-F 3 "https://www.mouser.de/ProductDetail/Yageo/RC0603FR-0759RL?qs=sGAEpiMZZMtlubZbdhIBIHvQf5egq9lvwCJIG56bzdE%3d" H 10350 6300 50  0001 C CNN
+F 3 "https://www.mouser.de/ProductDetail/Bourns/CR0603-FX-60R4ELF?qs=sGAEpiMZZMu61qfTUdNhG6LqqFhkr6pUa8gjAX4b5rM%3d" H 10350 6300 50  0001 C CNN
 	1    10350 6300
 	0    1    1    0

Commit message: crunch up 5v supply
Connections:
- net +BATT: now also J4.3 (Pin_3); no longer J4.1 (Pin_1)
- net CANH: now also J4.1 (Pin_1); no longer J4.3 (Pin_3)
- net CANL: now also J4.2 (Pin_2); no longer J4.4 (Pin_4)
- net GND: now also J4.4 (Pin_4); no longer J4.2 (Pin_2)

Commit message: add protection circuitry
Parts:
- added C14, C15, C16, C17: 100n, Capacitors_SMD:C_0603, symbol C
- added D1: SS14, Diodes_SMD:D_SMA_Handsoldering, symbol D
- added D2: SMLJ22A-Q, Diodes_SMD:D_SMC, symbol D_Zener
- added D3: PESD1CAN-U, TO_SOT_Packages_SMD:SOT-23, symbol D_TVS_x2_AAC
Connections:
- net +3V3: now also C16.1
- net +5V: now also C14.1, C17.1
- net +BATT: now also D1.2 (A); no longer C8.1, U2.2 (VIN), U2.3 (EN)
- net CANH: now also D3.1 (A1)
- net CANL: now also D3.2 (A2)
- net GND: now also C14.2, C15.2, C16.2, C17.2, D2.2 (A), D3.3 (common)
- new net: C15.1, C8.1, D1.1 (K), D2.1 (K), U2.2 (VIN), U2.3 (EN)
Other:
- moved on the sheet: C10, C11, C8, C9, L1, R10, R9, U2, U3

Commit message: sensibilize resistor values
Parts:
- R2, R4: value 60.4 -> 62
- R5, R6, R7: value 60.4 -> 100
Changed lines of the file:
@@
 P 7750 4500
 F 0 "R2" V 7830 4500 50  0000 C CNN
-F 1 "60.4" V 7750 4500 50  0000 C CNN
+F 1 "62" V 7750 4500 50  0000 C CNN
 F 2 "Resistors_SMD:R_0603" V 7680 4500 50  0001 C CNN
-F 3 "https://www.mouser.de/ProductDetail/Bourns/CR0603-FX-60R4ELF?qs=sGAEpiMZZMu61qfTUdNhG6LqqFhkr6pUa8gjAX4b5rM%3d" H 7750 4500 50  0001 C CNN
+F 3 "https://www.mouser.de/ProductDetail/Bourns/CR0603-FX-62R0ELF?qs=0nF2VnfAjXnEYbikTYe9aw%3d%3d" H 7750 4500 50  0001 C CNN
 	1    7750 4500
 	-1   0    0    1
@@
 P 7950 4500
 F 0 "R4" V 8030 4500 50  0000 C CNN
-F 1 "60.4" V 7950 4500 50  0000 C CNN
+F 1 "62" V 7950 4500 50  0000 C CNN
 F 2 "Resistors_SMD:R_0603" V 7880 4500 50  0001 C CNN
-F 3 "https://www.mouser.de/ProductDetail/Bourns/CR0603-FX-60R4ELF?qs=sGAEpiMZZMu61qfTUdNhG6LqqFhkr6pUa8gjAX4b5rM%3d" H 7950 4500 50  0001 C CNN
+F 3 "https://www.mouser.de/ProductDetail/Bourns/CR0603-FX-62R0ELF?qs=0nF2VnfAjXnEYbikTYe9aw%3d%3d" H 7950 4500 50  0001 C CNN
 	1    7950 4500
 	-1   0    0    1
@@
 P 10350 5900
 F 0 "R5" V 10430 5900 50  0000 C CNN
-F 1 "60.4" V 10350 5900 50  0000 C CNN
+F 1 "100" V 10350 5900 50  0000 C CNN
 F 2 "Resistors_SMD:R_0603" V 10280 5900 50  0001 C CNN
-F 3 "https://www.mouser.de/ProductDetail/Bourns/CR0603-FX-60R4ELF?qs=sGAEpiMZZMu61qfTUdNhG6LqqFhkr6pUa8gjAX4b5rM%3d" H 10350 5900 50  0001 C CNN
+F 3 "" H 10350 5900 50  0001 C CNN
 	1    10350 5900
 	0    -1   -1   0
@@
 P 10350 6000
 F 0 "R6" V 10430 6000 50  0000 C CNN
-F 1 "60.4" V 10350 6000 50  0000 C CNN
+F 1 "100" V 10350 6000 50  0000 C CNN
 F 2 "Resistors_SMD:R_0603" V 10280 6000 50  0001 C CNN
-F 3 "https://www.mouser.de/ProductDetail/Bourns/CR0603-FX-60R4ELF?qs=sGAEpiMZZMu61qfTUdNhG6LqqFhkr6pUa8gjAX4b5rM%3d" H 10350 6000 50  0001 C CNN
+F 3 "" H 10350 6000 50  0001 C CNN
 	1    10350 6000
 	0    1    1    0
@@
 P 10350 6300
 F 0 "R7" V 10430 6300 50  0000 C CNN
-F 1 "60.4" V 10350 6300 50  0000 C CNN
+F 1 "100" V 10350 6300 50  0000 C CNN
 F 2 "Resistors_SMD:R_0603" V 10280 6300 50  0001 C CNN
-F 3 "https://www.mouser.de/ProductDetail/Bourns/CR0603-FX-60R4ELF?qs=sGAEpiMZZMu61qfTUdNhG6LqqFhkr6pUa8gjAX4b5rM%3d" H 10350 6300 50  0001 C CNN
+F 3 "" H 10350 6300 50  0001 C CNN
 	1    10350 6300
 	0    1    1    0

Commit message: make 2 position slide switches instead of 4
Parts:
- SW1: footprint Buttons_Switches_THT:SW_DIP_x4_W7.62mm_Slide -> Buttons_Switches_THT:SW_DIP_x2_W7.62mm_Slide; symbol SW_DIP_x04 -> SW_DIP_x02
Connections:
- net at SW1.3: now also C7.1, SW1.4
Changed lines of the file:
@@
 $EndComp
 $Comp
-L SW_DIP_x04 SW1
+L SW_DIP_x02 SW1
 U 1 1 5AFC4E3D
-P 9900 4450
-F 0 "SW1" H 9900 4800 50  0000 C CNN
+P 9900 4350
+F 0 "SW1" H 9900 4600 50  0000 C CNN
 F 1 "CONFIG" H 9900 4200 50  0000 C CNN
-F 2 "Buttons_Switches_THT:SW_DIP_x4_W7.62mm_Slide" H 9900 4450 50  0001 C CNN
-F 3 "https://www.mouser.de/ProductDetail/TE-Connectivity-Alcoswitch/ADE0404?qs=sGAEpiMZZMv%2f%252b2JhlA6ysER62VlXw6iZ4HTlb4kKXdw%3d" H 9900 4450 50  0001 C CNN
-	1    9900 4450
+F 2 "Buttons_Switches_THT:SW_DIP_x2_W7.62mm_Slide" H 9900 4350 50  0001 C CNN
+F 3 "https://www.mouser.de/ProductDetail/Apem/NDS02V?qs=sGAEpiMZZMvHnN%252b%2fGH9WnarhEfYmPrhIFZ2OxET8b5I%3d" H 9900 4350 50  0001 C CNN
+	1    9900 4350
 	1    0    0    -1
 $EndComp
